File: NFC-Attendance-System.sch (EAGLE design)
At the start: 14 parts, among them J1 NFC_HDR, J2 DAC_HDR, J3 LCD_HDR, Q1 600mA/40V, SW1 PROG, SW2 RST, U1 ESP-WROOM-32

Commit message: minor fixes
Parts:
- Q1: value 600mA/40V -> 8550
Changed lines of the file:
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@@
 <part name="J3" library="SparkFun-Connectors" deviceset="CONN_08" device="&quot;" value="LCD_HDR"/>
 <part name="J2" library="SparkFun-Connectors" deviceset="CONN_07" device="" value="DAC_HDR"/>
-<part name="Q1" library="SparkFun-DiscreteSemi" deviceset="TRANS_PNP" device="-MMBT4403" value="600mA/40V"/>
+<part name="Q1" library="SparkFun-DiscreteSemi" deviceset="TRANS_PNP" device="-MMBT4403" value="8550"/>
 <part name="GND8" library="SparkFun-PowerSymbols" deviceset="GND" device=""/>
 <part name="FRAME1" library="SparkFun-Aesthetics" deviceset="FRAME-LETTER" device="">

Commit message: minor fixes
Parts:
- R3: value 5.1K -> 5.1k
- R4: value 1K -> 1k
Changed lines of the file:
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@@
 <drawing>
 <settings>
-<setting alwaysvectorfont="no"/>
+<setting alwaysvectorfont="yes"/>
 <setting keepoldvectorfont="yes"/>
 <setting verticaltext="up"/>
@@
 <schematic xreflabel="%F%N/%S.%C%R" xrefpart="/%S.%C%R">
 <attributes>
-<attribute name="CNAME" value="Jack Chen"/>
-<attribute name="REV" value="1"/>
 </attributes>
 <variantdefs>
@@
 <attribute name="REV" value="1.0"/>
 </part>
-<part name="R4" library="rcl" library_urn="urn:adsk.eagle:library:334" deviceset="R-EU_" device="R0603" package3d_urn="urn:adsk.eagle:package:23555/3" value="1K"/>
-<part name="R3" library="rcl" library_urn="urn:adsk.eagle:library:334" deviceset="R-EU_" device="R0603" package3d_urn="urn:adsk.eagle:package:23555/3" value="5.1K"/>
+<part name="R4" library="rcl" library_urn="urn:adsk.eagle:library:334" deviceset="R-EU_" device="R0603" package3d_urn="urn:adsk.eagle:package:23555/3" value="1k"/>
+<part name="R3" library="rcl" library_urn="urn:adsk.eagle:library:334" deviceset="R-EU_" device="R0603" package3d_urn="urn:adsk.eagle:package:23555/3" value="5.1k"/>
 <part name="SUPPLY2" library="supply2" library_urn="urn:adsk.eagle:library:372" deviceset="+5V" device=""/>
 </parts>

Commit message: minor fixes
Parts:
- added R5, R6, R7: 1k, rcl:R-EU_R0603
Connections:
- new net N$2: Q1.B, R4.2
- net +5V: now also R6.2; no longer R4.2
- net GND: now also R5.1, R7.1
- net LCD_BL: now also R7.2
- net PN532_RST: now also R4.1, R5.2; no longer Q1.B
- net RSTPD_N: now also R6.1; no longer R4.1
Other:
- moved on the sheet: J1, Q1, R4
